Commit message: Refactor robotic_actor to implement reservoir gate control and update URDF model for new structure

File: robotic_actor/urdf/four_bar.urdf (robot description, URDF)
Before this commit: robot four_bar_linkage, 4 links, 4 joints
Links:
- removed link coupler
- removed link link1
- removed link link2
- added link gate, mass 0.3; collision box size=0.56 0.56 0.04; visual box size=0.56 0.56 0.04
- added link wall_back, mass 0.1; collision box size=0.6 0.02 0.3; visual box size=0.6 0.02 0.3
- added link wall_front, mass 0.1; collision box size=0.6 0.02 0.3; visual box size=0.6 0.02 0.3
- added link wall_left, mass 0.1; collision box size=0.02 0.56 0.3; visual box size=0.02 0.56 0.3
- link base_link: mass 0.1 -> 0.5; geometry collision box size=0.6 0.6 0.02; visual box size=0.6 0.6 0.02
Joints:
- removed joint joint1
- removed joint joint2
- removed joint joint3
- removed joint joint4
- added joint gate_joint: type revolute, parent base_link, child gate, origin xyz=0 0.28 0.3 rpy=0 0 0, axis 1 0 0, limit lower=0 upper=1.57 effort=10 velocity=2.0
- added joint wall_back_joint: type fixed, parent base_link, child wall_back, origin xyz=0 0.29 0 rpy=0 0 0
- added joint wall_front_joint: type fixed, parent base_link, child wall_front, origin xyz=0 -0.29 0 rpy=0 0 0
- added joint wall_left_joint: type fixed, parent base_link, child wall_left, origin xyz=-0.29 0 0 rpy=0 0 0
