Commit message: Add TCP joint and tool link to URDF model; include tcp_monitor.py script in installation

File: robot_arm/urdf/mybot.urdf.xacro (robot description, xacro)
@@ -235,4 +235,29 @@
 		<child link="right_gripper_finger"/>
 	</joint>
+	<!-- TCP frames -->
+	<joint name="tool0_joint" type="fixed">
+		<origin xyz="0 0 0.025" rpy="0 0 0"/>
+		<parent link="hand"/>
+		<child link="tool0"/>
+	</joint>
+	<link name="tool0"/>
+	<joint name="tcp_joint" type="fixed">
+		<origin xyz="0 0 0.045" rpy="0 0 0"/>
+		<parent link="tool0"/>
+		<child link="tcp"/>
+	</joint>
+	<link name="tcp">
+		<visual>
+			<geometry>
+				<sphere radius="0.01"/>
+			</geometry>
+			<material name="tcp_red">
+				<color rgba="1 0 0 1"/>
+			</material>
+		</visual>
+	</link>
+	<gazebo reference="tcp">
+		<material>Gazebo/Red</material>
+	</gazebo>
 	<!-- ==================== ros2_control ==================== -->
 	<ros2_control name="robot_arm_control" type="system">

Commit message: Add cotton_field world to simulation and update launch file to use it. Adjusted inertia values in URDF for left and right gripper bases for physical consistency.

File: robot_arm/urdf/mybot.urdf.xacro (robot description, xacro)
@@ -143,5 +143,6 @@
 		<inertial>
 			<mass value="0.01"/>
-			<inertia ixx="8.23e-8" iyy="8.23e-8" izz="3.47e-7" ixy="0" ixz="0" iyz="0"/>
+			<!-- Box approx: 0.005 x 0.005 x 0.02 (see visual). Keep inertia physically consistent. -->
+			<inertia ixx="3.54e-7" iyy="3.54e-7" izz="4.17e-8" ixy="0" ixz="0" iyz="0"/>
 		</inertial>
 		<visual>
@@ -168,5 +169,6 @@
 		<inertial>
 			<mass value="0.01"/>
-			<inertia ixx="8.23e-8" iyy="8.23e-8" izz="3.47e-7" ixy="0" ixz="0" iyz="0"/>
+			<!-- Box approx: 0.005 x 0.005 x 0.02 (see visual). Keep inertia physically consistent. -->
+			<inertia ixx="3.54e-7" iyy="3.54e-7" izz="4.17e-8" ixy="0" ixz="0" iyz="0"/>
 		</inertial>
 		<visual>

Commit message: Add environment configuration and landmark publisher for robotic arm simulation
- Introduced `environment_config.yaml` as a single source of truth for landmark positions and exploration parameters.
- Added `landmark_publisher.py` to publish static TF frames and collision objects for MoveIt.
- Updated launch files to integrate the landmark publisher and ensure proper initialization order.
- Enhanced `cotton_field.world` with visual markers for exploration start and end points.
- Adjusted installation scripts to include new configuration and publisher files.

File: robot_arm/urdf/mybot.urdf.xacro (robot description, xacro)
@@ -1,4 +1,6 @@
 <?xml version="1.0"?>
 <robot xmlns:xacro="http://www.ros.org/wiki/xacro" name="arm">
+	<!-- Xacro arguments (injected from launch file) -->
+	<xacro:arg name="controllers_yaml" default=""/>
 	<!-- World link (fixed reference) -->
 	<link name="world"/>
@@ -262,4 +264,77 @@
 		<material>Gazebo/Red</material>
 	</gazebo>
+	<!-- ==================== Wrist-Mounted Camera ==================== -->
+	<!-- Camera link attached to tool0, offset to avoid gripper clipping -->
+	<joint name="camera_joint" type="fixed">
+		<parent link="tool0"/>
+		<child link="camera_link"/>
+		<origin xyz="0.02 0 0.01" rpy="0 0.3 0"/>  <!-- Slightly forward and tilted down -->
+	</joint>
+	<link name="camera_link">
+		<visual>
+			<geometry>
+				<box size="0.02 0.03 0.02"/>
+			</geometry>
+			<material name="camera_black">
+				<color rgba="0.1 0.1 0.1 1"/>
+			</material>
+		</visual>
+		<collision>
+			<geometry>
+				<box size="0.02 0.03 0.02"/>
+			</geometry>
+		</collision>
+		<inertial>
+			<mass value="0.05"/>
+			<inertia ixx="1e-6" iyy="1e-6" izz="1e-6" ixy="0" ixz="0" iyz="0"/>
+		</inertial>
+	</link>
+	<!-- ROS optical frame convention: Z forward, X right, Y down -->
+	<joint name="camera_optical_joint" type="fixed">
+		<parent link="camera_link"/>
+		<child link="camera_optical_frame"/>
+		<origin xyz="0 0 0" rpy="-1.5708 0 -1.5708"/>
+	</joint>
+	<link name="camera_optical_frame"/>
+	<!-- Gazebo camera (material + RGB-D sensor) -->
+	<gazebo reference="camera_link">
+		<material>Gazebo/Black</material>
+		<sensor type="depth" name="wrist_rgbd_camera">
+			<always_on>true</always_on>
+			<update_rate>30.0</update_rate>
+			<camera name="wrist_camera">
+				<horizontal_fov>1.047</horizontal_fov>
+				<image>
+					<width>640</width>
+					<height>480</height>
+					<format>R8G8B8</format>
+				</image>
+				<clip>
+					<near>0.05</near>
+					<far>3.0</far>
+				</clip>
+				<noise>
+					<type>gaussian</type>
+					<mean>0.0</mean>
+					<stddev>0.007</stddev>
+				</noise>
+			</camera>
+			<plugin name="camera_plugin" filename="libgazebo_ros_camera.so">
+				<ros>
+					<namespace>/camera</namespace>
+					<remapping>image_raw:=color/image_raw</remapping>
+					<remapping>camera_info:=color/camera_info</remapping>
+					<remapping>depth/image_raw:=depth/image_raw</remapping>
+					<remapping>depth/camera_info:=depth/camera_info</remapping>
+					<remapping>points:=depth/points</remapping>
+				</ros>
+				<camera_name>wrist</camera_name>
+				<frame_name>camera_optical_frame</frame_name>
+				<hack_baseline>0.07</hack_baseline>
+				<min_depth>0.05</min_depth>
+				<max_depth>3.0</max_depth>
+			</plugin>
+		</sensor>
+	</gazebo>
 	<!-- ==================== ros2_control ==================== -->
 	<ros2_control name="robot_arm_control" type="system">
@@ -319,7 +394,5 @@
 	<gazebo>
 		<plugin filename="libgazebo_ros2_control.so" name="gazebo_ros2_control">
-			<robot_param>robot_description</robot_param>
-			<robot_param_node>robot_state_publisher</robot_param_node>
-			<parameters>$(find robot_arm)/yaml/controllers.yaml</parameters>
+			<parameters>$(arg controllers_yaml)</parameters>
 		</plugin>
 	</gazebo>

Commit message: Update URDF and SRDF configurations for robotic arm
- Added collision geometry for the TCP link in the URDF to enhance simulation accuracy.
- Refactored the arm planning group in the SRDF to use a chain structure instead of individual joints, streamlining the configuration.

File: robot_arm/urdf/mybot.urdf.xacro (robot description, xacro)
@@ -260,4 +260,9 @@
 			</material>
 		</visual>
+		<collision>
+			<geometry>
+				<sphere radius="0.01"/>
+			</geometry>
+		</collision>
 	</link>
 	<gazebo reference="tcp">

Commit message: Add exploration commands and update environment configuration
- Introduced a new `commands.md` file with essential commands for building and launching the robot arm and its configurations.
- Adjusted exploration path endpoints in `environment_config.yaml` for improved camera stability and reachability.
- Updated the URDF to reposition the camera link for a better view and modified the exploration markers in `cotton_field.world` to match the new configurations.
- Enhanced `arm_commander.py` to include orientation constraints for the camera during exploration, ensuring stable viewing angles.

File: robot_arm/urdf/mybot.urdf.xacro (robot description, xacro)
@@ -270,9 +270,11 @@
 	</gazebo>
 	<!-- ==================== Wrist-Mounted Camera ==================== -->
-	<!-- Camera link attached to tool0, offset to avoid gripper clipping -->
+	<!-- Camera link attached to lower_arm (forearm), providing a stable view -->
 	<joint name="camera_joint" type="fixed">
-		<parent link="tool0"/>
+		<parent link="lower_arm"/>
 		<child link="camera_link"/>
-		<origin xyz="0.02 0 0.01" rpy="0 0.3 0"/>  <!-- Slightly forward and tilted down -->
+		<!-- Position: On "top" of the lower_arm (Negative X based on visual feedback), near the end -->
+		<!-- Orientation: Pitch -90 (-1.57) to point forward along the arm -->
+		<origin xyz="-0.08 0.0 0.35" rpy="0 -1.57 0"/>
 	</joint>
 	<link name="camera_link">

Commit message: Refactor explorer node for circular arc sweep exploration
- Updated the `explorer.py` to implement a circular arc sweep method for cluster detection, replacing the previous mini-sweep approach.
- Enhanced viewpoint generation to include multiple angles around each cluster, improving detection robustness.
- Adjusted parameters for arc angle, number of views per cluster, and height variation to optimize scanning.
- Modified logging to reflect the new scanning strategy and provide detailed viewpoint information during execution.
- Updated URDF to reposition the camera for better alignment with the gripper.

File: robot_arm/urdf/mybot.urdf.xacro (robot description, xacro)
@@ -270,11 +270,11 @@
 	</gazebo>
 	<!-- ==================== Wrist-Mounted Camera ==================== -->
-	<!-- Camera link attached to lower_arm (forearm), providing a stable view -->
+	<!-- Camera link attached to tool0 - camera looks same direction as gripper -->
+	<!-- Gazebo camera looks along +X of sensor link, so rotate to align with tool0 +Z -->
 	<joint name="camera_joint" type="fixed">
-		<parent link="lower_arm"/>
+		<parent link="tool0"/>
 		<child link="camera_link"/>
-		<!-- Position: On "top" of the lower_arm (Negative X based on visual feedback), near the end -->
-		<!-- Orientation: Pitch -90 (-1.57) to point forward along the arm -->
-		<origin xyz="-0.08 0.0 0.35" rpy="0 -1.57 0"/>
+		<!-- Position: Above gripper (-X), Rotation: -90° pitch so camera X aligns with tool0 Z -->
+		<origin xyz="-0.04 0 0" rpy="0 -1.5708 0"/>
 	</joint>
 	<link name="camera_link">

Commit message: Add migration guide for Gazebo Classic to Gazebo Sim and update robot_arm configurations
- Introduced a comprehensive migration guide detailing the transition from Gazebo Classic to Gazebo Sim, including version compatibility and necessary changes.
- Updated `package.xml` to replace dependencies for Gazebo Classic with those for Gazebo Sim.
- Created `gz_bridge.yaml` for ROS-Gazebo bridge configuration.
- Modified `bot.launch.py` to launch the robot in Gazebo Sim, incorporating new bridge nodes for topic communication.
- Updated URDF files to reflect changes in sensor plugins and control interfaces for Gazebo Sim.
- Enhanced the `cotton_field.world` file with required plugins and lighting adjustments for Gazebo Sim compatibility.
- Added commands for building the harvester interfaces alongside existing packages.

File: robot_arm/urdf/mybot.urdf.xacro (robot description, xacro)
@@ -266,7 +266,5 @@
 		</collision>
 	</link>
-	<gazebo reference="tcp">
-		<material>Gazebo/Red</material>
-	</gazebo>
+	<!-- TCP uses material from URDF visual (tcp_red) -->
 	<!-- ==================== Wrist-Mounted Camera ==================== -->
 	<!-- Camera link attached to tool0 - camera looks same direction as gripper -->
@@ -304,10 +302,11 @@
 	</joint>
 	<link name="camera_optical_frame"/>
-	<!-- Gazebo camera (material + RGB-D sensor) -->
+	<!-- Gazebo Sim camera (RGB-D sensor - generic, ROS bridge handles communication) -->
 	<gazebo reference="camera_link">
-		<material>Gazebo/Black</material>
-		<sensor type="depth" name="wrist_rgbd_camera">
+		<sensor type="rgbd_camera" name="wrist_rgbd_camera">
 			<always_on>true</always_on>
 			<update_rate>30.0</update_rate>
+			<topic>camera</topic>
+			<ignition_frame_id>camera_optical_frame</ignition_frame_id>
 			<camera name="wrist_camera">
 				<horizontal_fov>1.047</horizontal_fov>
@@ -321,4 +320,10 @@
 					<far>3.0</far>
 				</clip>
+				<depth_camera>
+					<clip>
+						<near>0.05</near>
+						<far>3.0</far>
+					</clip>
+				</depth_camera>
 				<noise>
 					<type>gaussian</type>
@@ -327,19 +332,4 @@
 				</noise>
 			</camera>
-			<plugin name="camera_plugin" filename="libgazebo_ros_camera.so">
-				<ros>
-					<namespace>/camera</namespace>
-					<remapping>image_raw:=color/image_raw</remapping>
-					<remapping>camera_info:=color/camera_info</remapping>
-					<remapping>depth/image_raw:=depth/image_raw</remapping>
-					<remapping>depth/camera_info:=depth/camera_info</remapping>
-					<remapping>points:=depth/points</remapping>
-				</ros>
-				<camera_name>wrist</camera_name>
-				<frame_name>camera_optical_frame</frame_name>
-				<hack_baseline>0.07</hack_baseline>
-				<min_depth>0.05</min_depth>
-				<max_depth>3.0</max_depth>
-			</plugin>
 		</sensor>
 	</gazebo>
@@ -347,5 +337,5 @@
 	<ros2_control name="robot_arm_control" type="system">
 		<hardware>
-			<plugin>gazebo_ros2_control/GazeboSystem</plugin>
+			<plugin>ign_ros2_control/IgnitionSystem</plugin>
 		</hardware>
 		<joint name="hip">
@@ -398,37 +388,11 @@
 		</joint>
 	</ros2_control>
-	<!-- ==================== Gazebo ROS2 Control Plugin ==================== -->
+	<!-- ==================== Gazebo Sim ROS2 Control Plugin (Ignition Fortress) ==================== -->
 	<gazebo>
-		<plugin filename="libgazebo_ros2_control.so" name="gazebo_ros2_control">
+		<plugin filename="ign_ros2_control-system" name="ign_ros2_control::IgnitionROS2ControlPlugin">
 			<parameters>$(arg controllers_yaml)</parameters>
 		</plugin>
 	</gazebo>
-	<!-- Gazebo material colors -->
-	<gazebo reference="base_link">
-		<material>Gazebo/Grey</material>
-	</gazebo>
-	<gazebo reference="torso">
-		<material>Gazebo/Grey</material>
-	</gazebo>
-	<gazebo reference="upper_arm">
-		<material>Gazebo/Grey</material>
-	</gazebo>
-	<gazebo reference="lower_arm">
-		<material>Gazebo/Grey</material>
-	</gazebo>
-	<gazebo reference="hand">
-		<material>Gazebo/Grey</material>
-	</gazebo>
-	<gazebo reference="left_gripper_base">
-		<material>Gazebo/Grey</material>
-	</gazebo>
-	<gazebo reference="right_gripper_base">
-		<material>Gazebo/Grey</material>
-	</gazebo>
-	<gazebo reference="left_gripper_finger">
-		<material>Gazebo/Grey</material>
-	</gazebo>
-	<gazebo reference="right_gripper_finger">
-		<material>Gazebo/Grey</material>
-	</gazebo>
+	<!-- Note: Gazebo Sim uses materials from URDF visuals directly -->
+	<!-- Old Gazebo/Grey references removed - not needed in Ignition -->
 </robot>

Commit message: Update explorer node and URDF for enhanced scanning and joint limits
- Modified the `ExplorerNode` class to support three rows of camera positions for panoramic scanning, improving coverage.
- Adjusted dynamic row naming logic to accommodate the new configuration.
- Updated elbow joint limits in the URDF to allow for a wider range of motion, enhancing arm flexibility during operations.

File: robot_arm/urdf/mybot.urdf.xacro (robot description, xacro)
@@ -112,5 +112,5 @@
 	<joint name="elbow" type="revolute">
 		<axis xyz="0 1 0"/>
-		<limit velocity="1.0" effort="30.0" upper="1.5708" lower="-1.5708"/>
+		<limit velocity="1.0" effort="30.0" upper="2.1" lower="-2.1"/>
 		<parent link="upper_arm"/>
 		<child link="lower_arm"/>
@@ -357,6 +357,6 @@
 		<joint name="elbow">
 			<command_interface name="position">
-				<param name="min">-1.5708</param>
-				<param name="max">1.5708</param>
+				<param name="min">-2.1</param>
+				<param name="max">2.1</param>
 			</command_interface>
 			<state_interface name="position"/>

Commit message: Update documentation and figures for RoboCot project
- Replaced mock YOLO detector command with real YOLO detector in `commands.md`.
- Added new figures: `cluster_with_unripe_bolls.png`, `cluster_with_unripe_bolls_old.png`, and `figure_12_visual_servoing_convergence.svg` to enhance visual documentation.
- Introduced `generate_visual_servoing_figure.py` script to automate the creation of the visual servoing convergence figure.
- Updated `preview_figures.html` to include new figures for better accessibility.
- Enhanced YOLO static image processing with `run_yolo_static.py` for improved detection capabilities.
- Adjusted spatial detection pipeline to utilize cluster detection services, refining detection accuracy and logging.
- Updated URDF for the robot arm to specify joint limits for improved control.

File: robot_arm/urdf/mybot.urdf.xacro (robot description, xacro)
@@ -55,6 +55,7 @@
 		</collision>
 	</link>
-	<joint name="hip" type="continuous">
+	<joint name="hip" type="revolute">
 		<axis xyz="0 0 1"/>
+		<limit velocity="1.0" effort="30.0" lower="-3.14159" upper="3.14159"/>
 		<parent link="base_link"/>
 		<child link="torso"/>
@@ -135,6 +136,7 @@
 		</collision>
 	</link>
-	<joint name="wrist" type="continuous">
+	<joint name="wrist" type="revolute">
 		<axis xyz="0 1 0"/>
+		<limit velocity="1.0" effort="30.0" lower="-3.14159" upper="3.14159"/>
 		<parent link="lower_arm"/>
 		<child link="hand"/>
