Commit message: Current approach: IK → joint goal → OMPL plans joint-space path → execute collision avoidance yok.
Enhance task documentation and robot arm configurations

- Updated `tasks_today.md` to include a detailed overview of existing components and missing elements for the pick-and-place functionality, outlining necessary steps for implementation.
- Modified `camera_focus.py` to increase velocity and acceleration scaling factors for improved performance.
- Adjusted `bot.launch.py` to set the robot's initial z-position to 0.0 for better alignment with the simulation environment.
- Revised `m1013_robocot.urdf.xacro` to ensure consistency in the robot's base pose and updated camera settings for optimal performance.
- Added dynamic cotton bolls to `cotton_field.world` to facilitate grasping during simulations.
- Updated `ompl_planning.yaml` to change the default planner to RRTstar for enhanced path planning capabilities.
- Refactored `arm_commander.py` to implement IK for target poses, improving the robot's movement reliability and efficiency.

File: robot_arm/urdf/m1013_robocot.urdf.xacro (robot description, xacro)
@@ -12,6 +12,7 @@
 	<!-- ==================== World ==================== -->
 	<link name="world"/>
+	<!-- Must match bot.launch.py spawn (-z 0.1): TF world == Gazebo world for base pose -->
 	<joint name="world_fixed" type="fixed">
-		<origin xyz="0 0 0" rpy="0 0 0"/>
+		<origin xyz="0 0 0.1" rpy="0 0 0"/>
 		<parent link="world"/>
 		<child link="base_0"/>
@@ -399,5 +400,5 @@
 		<sensor type="rgbd_camera" name="wrist_rgbd_camera">
 			<always_on>true</always_on>
-			<update_rate>30.0</update_rate>
+			<update_rate>1.0</update_rate>
 			<topic>camera</topic>
 			<ignition_frame_id>camera_optical_frame</ignition_frame_id>

Commit message: Enhance gripper functionality and update documentation
- Modified `gripper_controller.py` to support both left and right finger joints for improved gripper control.
- Updated `m1013_robocot.urdf.xacro` to define the right finger joint, ensuring accurate simulation and control.
- Adjusted `controllers.yaml` to include the right finger joint in the gripper controller configuration.
- Expanded `tasks_today.md` to clarify the simulation and real-world behavior of the gripper, detailing the differences in feedback mechanisms.

File: robot_arm/urdf/m1013_robocot.urdf.xacro (robot description, xacro)
@@ -322,5 +322,4 @@
 		<axis xyz="1 0 0"/>
 		<limit effort="130" lower="0" upper="0.025" velocity="0.15"/>
-		<mimic joint="hande_left_finger_joint" multiplier="1" offset="0"/>
 	</joint>
 	<link name="hande_right_finger">
@@ -506,6 +505,14 @@
 			<state_interface name="velocity"/>
 		</joint>
-		<!-- Gripper joint (prismatic) -->
+		<!-- Gripper joints (prismatic) -->
 		<joint name="hande_left_finger_joint">
+			<command_interface name="position">
+				<param name="min">0</param>
+				<param name="max">0.025</param>
+			</command_interface>
+			<state_interface name="position"/>
+			<state_interface name="velocity"/>
+		</joint>
+		<joint name="hande_right_finger_joint">
 			<command_interface name="position">
 				<param name="min">0</param>

Commit message: Update joint configurations and enhance arm commander functionality
- Adjusted joint5 range in `harvest_pipeline.launch.py` and `robot_arm_moveit_config/config/robot_arm.srdf` to improve arm positioning.
- Updated home joint values in `explorer.py` and `arm_commander.py` for consistency across modules.
- Enhanced `arm_commander.py` with new services for rotating the wrist joint (joint5) and improved logging for home position movements.

File: robot_arm/urdf/m1013_robocot.urdf.xacro (robot description, xacro)
@@ -367,10 +367,12 @@
 		<parent link="link6"/>
 		<child link="camera_link"/>
-		<origin xyz="-0.05 0 -0.02" rpy="0 -1.5708 0"/>
+		<!-- Camera +X (Gazebo look direction) aligned with link6 +Z (approach direction) -->
+		<!-- X=-0.08: far back from gripper, Z=-0.02: slight side offset -->
+		<origin xyz="-0.14 0 -0.02" rpy="0 -1.5708 0"/>
 	</joint>
 	<link name="camera_link">
 		<visual>
 			<geometry>
-				<box size="0.02 0.03 0.02"/>
+				<box size="0.06 0.09 0.06"/>
 			</geometry>
 			<material name="camera_black">
@@ -378,7 +380,17 @@
 			</material>
 		</visual>
-		<collision>
-			<geometry>
-				<box size="0.02 0.03 0.02"/>
+		<!-- Mounting arm connecting camera back to link6 -->
+		<visual>
+			<origin xyz="0.01 0 -0.07" rpy="0 0 0"/>
+			<geometry>
+				<cylinder radius="0.012" length="0.14"/>
+			</geometry>
+			<material name="camera_mount_grey">
+				<color rgba="0.4 0.4 0.4 1"/>
+			</material>
+		</visual>
+		<collision>
+			<geometry>
+				<box size="0.06 0.09 0.06"/>
 			</geometry>
 		</collision>
@@ -399,5 +411,5 @@
 		<sensor type="rgbd_camera" name="wrist_rgbd_camera">
 			<always_on>true</always_on>
-			<update_rate>1.0</update_rate>
+			<update_rate>30.0</update_rate>
 			<topic>camera</topic>
 			<ignition_frame_id>camera_optical_frame</ignition_frame_id>

Commit message: Refactor RoboCot project documentation and enhance harvest log parsing
- Updated `CHECKPOINT.md` to reflect the current project status and repository structure, including detailed descriptions of the cotton harvesting robot and its capabilities.
- Introduced `parse_harvest_log.py` to parse and summarize harvest pipeline logs, extracting critical information for easier analysis.
- Adjusted joint configurations in `harvest_pipeline.launch.py` and `explorer.py` to improve arm positioning and consistency.
- Enhanced `gripper_controller.py` to support only the left finger joint, with the right finger following via a mimic tag, streamlining gripper control.
- Updated various files to improve logging and functionality in the harvesting process, ensuring better tracking and performance metrics.

File: robot_arm/urdf/m1013_robocot.urdf.xacro (robot description, xacro)
@@ -315,5 +315,5 @@
 		</collision>
 	</link>
-	<!-- Right finger (mimic of left) -->
+	<!-- Right finger (mimic of left — Gazebo drives this automatically) -->
 	<joint name="hande_right_finger_joint" type="prismatic">
 		<parent link="hand_e_link"/>
@@ -322,4 +322,5 @@
 		<axis xyz="1 0 0"/>
 		<limit effort="130" lower="0" upper="0.025" velocity="0.15"/>
+		<mimic joint="hande_left_finger_joint" multiplier="1.0" offset="0.0"/>
 	</joint>
 	<link name="hande_right_finger">
@@ -526,12 +527,5 @@
 			<state_interface name="velocity"/>
 		</joint>
-		<joint name="hande_right_finger_joint">
-			<command_interface name="position">
-				<param name="min">0</param>
-				<param name="max">0.025</param>
-			</command_interface>
-			<state_interface name="position"/>
-			<state_interface name="velocity"/>
-		</joint>
+		<!-- hande_right_finger_joint: mimic of left, driven by Gazebo physics (no ros2_control interface) -->
 	</ros2_control>
 	<!-- ==================== Gazebo Sim ROS2 Control Plugin ==================== -->

Commit message: Add Husky robot launch and URDF files for orchard simulation
- Introduced husky_test.launch.py to spawn the Husky robot with M1013 and reservoir in the orchard world, enabling a F1.4 sanity check for URDF composition.
- Created husky_robocot.urdf.xacro to define the Husky robot's structure, including its body, wheels, arm mount, and reservoir.
- Updated m1013_robocot.urdf.xacro to support integration with the Husky platform by allowing for a non-standalone configuration.
- Enhanced the launch file to include necessary nodes for simulation, state publishing, and controller management, ensuring a comprehensive testing environment for the robot.

File: robot_arm/urdf/m1013_robocot.urdf.xacro (robot description, xacro)
@@ -10,12 +10,17 @@
 <robot xmlns:xacro="http://www.ros.org/wiki/xacro" name="m1013_robocot">
 	<xacro:arg name="controllers_yaml" default=""/>
-	<!-- ==================== World ==================== -->
-	<link name="world"/>
-	<!-- Must match bot.launch.py spawn (-z 0.1): TF world == Gazebo world for base pose -->
-	<joint name="world_fixed" type="fixed">
-		<origin xyz="0 0 0.1" rpy="0 0 0"/>
-		<parent link="world"/>
-		<child link="base_0"/>
-	</joint>
+	<!-- standalone=true: arm sits on its own at world (orchard_test, sim demo)
+	     standalone=false: arm is attached to a parent (Husky deck) by the
+	     including URDF, which defines its own world/base joint. -->
+	<xacro:arg name="standalone" default="true"/>
+	<!-- ==================== Standalone-only world fixture ==================== -->
+	<xacro:if value="$(arg standalone)">
+		<link name="world"/>
+		<joint name="world_fixed" type="fixed">
+			<origin xyz="0 0 0.1" rpy="0 0 0"/>
+			<parent link="world"/>
+			<child link="base_0"/>
+		</joint>
+	</xacro:if>
 	<!-- ==================== M1013 Arm ==================== -->
 	<!-- Base (link0) -->

Commit message: Refactor Gripper Controller and Update URDF for Simple Box Gripper
- Updated the Gripper Controller to support a new simple box gripper design, replacing the Robotiq Hand-E.
- Modified the gripper's parameters, including open and close positions, and implemented a more robust success reporting mechanism.
- Enhanced the URDF to reflect the new gripper structure, including a fixed right finger and a prismatic left finger with updated dimensions and physics properties.
- Adjusted the YAML and MoveIt configuration files to align with the new gripper design, ensuring proper integration with the control system.
- Improved the SimpleClusterHarvester to visually command the gripper open/close actions during the harvesting process, enhancing user feedback in simulation.

File: robot_arm/urdf/m1013_robocot.urdf.xacro (robot description, xacro)
@@ -255,6 +255,12 @@
 	</joint>
 	<link name="tool0"/>
-	<!-- ==================== Robotiq Hand-E Gripper ==================== -->
-	<!-- Fixed mount: Hand-E base attaches to tool0 (tool flange) -->
+	<!-- ==================== Simple Box Gripper ==================== -->
+	<!-- Robotiq Hand-E was replaced by a from-scratch minimal design:
+	     - Palm: dark box plate attached to tool0 (where Hand-E base was).
+	     - Right finger: thin grey prism, FIXED on the +X side of the palm.
+	     - Left finger:  thin grey prism, prismatic joint along +X. Slides
+	       between OPEN (-X end) and CLOSED (meets right pad at center).
+	     Single moving joint = guaranteed to work; no mesh, no mimic, no
+	     fancy physics. -->
 	<joint name="robotiq_hande_base_joint" type="fixed">
 		<parent link="tool0"/>
@@ -262,92 +268,78 @@
 		<origin xyz="0 0 0" rpy="0 0 0"/>
 	</joint>
+	<!-- Palm: thin plate, ~6cm wide (X), ~4cm deep (Y), 5cm tall (Z).
+	     Spans Z = 0 .. 0.05 from tool0. -->
 	<link name="hand_e_link">
 		<inertial>
-			<origin rpy="0 0 0" xyz="0 0 0.04607"/>
-			<mass value="0.86387"/>
-			<inertia ixx="1.01756e-03" ixy="0" ixz="2.235e-06" iyy="1.028041e-03" iyz="0" izz="4.8981e-04"/>
-		</inertial>
-		<visual>
-			<origin rpy="0 0 0" xyz="0 0 0"/>
-			<geometry>
-				<mesh filename="package://robot_arm/meshes/hande/hande.dae" scale="1.0 1.0 1.0"/>
-			</geometry>
-			<material name="HandE_Dark">
-				<color rgba="0.1 0.1 0.1 1.0"/>
+			<origin rpy="0 0 0" xyz="0 0 0.025"/>
+			<mass value="0.3"/>
+			<inertia ixx="0.0005" ixy="0" ixz="0" iyy="0.0005" iyz="0" izz="0.0005"/>
+		</inertial>
+		<visual>
+			<origin rpy="0 0 0" xyz="0 0 0.025"/>
+			<geometry>
+				<box size="0.060 0.040 0.050"/>
+			</geometry>
+			<material name="GripperPalm">
+				<color rgba="0.15 0.15 0.15 1.0"/>
 			</material>
 		</visual>
-		<visual>
-			<origin rpy="0 0 0" xyz="0 0 -0.0015"/>
-			<geometry>
-				<mesh filename="package://robot_arm/meshes/exchanger/hande_base.dae" scale="1.0 1.0 1.0"/>
-			</geometry>
-		</visual>
-		<collision>
-			<origin rpy="0 0 0" xyz="0 0 0"/>
-			<geometry>
-				<mesh filename="package://robot_arm/meshes/hande/hande-collision.dae" scale="1.0 1.0 1.0"/>
-			</geometry>
-		</collision>
-	</link>
-	<!-- Left finger (driven) -->
+		<collision>
+			<origin rpy="0 0 0" xyz="0 0 0.025"/>
+			<geometry>
+				<box size="0.060 0.040 0.050"/>
+			</geometry>
+		</collision>
+	</link>
+	<!-- Right finger: FIXED on +X side. Pad spans X: +0.015 .. +0.025,
+	     Z: 0.050 .. 0.130. -->
+	<joint name="hande_right_finger_joint" type="fixed">
+		<parent link="hand_e_link"/>
+		<child link="hande_right_finger"/>
+		<origin rpy="0 0 0" xyz="0.020 0 0.090"/>
+	</joint>
+	<link name="hande_right_finger">
+		<inertial>
+			<origin rpy="0 0 0" xyz="0 0 0"/>
+			<mass value="0.02"/>
+			<inertia ixx="1e-05" ixy="0" ixz="0" iyy="1e-05" iyz="0" izz="1e-05"/>
+		</inertial>
+		<visual>
+			<origin rpy="0 0 0" xyz="0 0 0"/>
+			<geometry>
+				<box size="0.010 0.025 0.080"/>
+			</geometry>
+			<material name="GripperFinger">
+				<color rgba="0.55 0.55 0.55 1.0"/>
+			</material>
+		</visual>
+	</link>
+	<!-- Left finger: PRISMATIC, single moving joint of the gripper.
+	     Joint origin sits at the OPEN pose (-0.020 X). Axis +X.
+	     - joint = 0     → link at (-0.020, 0, 0.090): pad spans X -0.025..-0.015 → OPEN, ~30mm gap
+	     - joint = 0.030 → link at (+0.010, 0, 0.090): pad spans X +0.005..+0.015 → CLOSED, touching right pad inner face -->
 	<joint name="hande_left_finger_joint" type="prismatic">
 		<parent link="hand_e_link"/>
 		<child link="hande_left_finger"/>
-		<origin rpy="0 0 0" xyz="0 0 0.099"/>
-		<axis xyz="-1 0 0"/>
-		<limit effort="130" lower="0" upper="0.025" velocity="0.15"/>
+		<origin rpy="0 0 0" xyz="-0.020 0 0.090"/>
+		<axis xyz="1 0 0"/>
+		<limit effort="100" lower="0.0" upper="0.030" velocity="1.0"/>
+		<dynamics damping="0.0" friction="0.0"/>
 	</joint>
 	<link name="hande_left_finger">
 		<inertial>
-			<origin rpy="0 0 0" xyz="0.02262 -0.00759 0.00738"/>
-			<mass value="0.05"/>
-			<inertia ixx="1e-04" ixy="0" ixz="0" iyy="1e-04" iyz="0" izz="1e-04"/>
-		</inertial>
-		<visual>
-			<origin rpy="0 0 0" xyz="0 0 0"/>
-			<geometry>
-				<mesh filename="package://robot_arm/meshes/hande/finger_1.dae" scale="1.0 1.0 1.0"/>
-			</geometry>
-			<material name="HandE_Gray">
-				<color rgba="0.4 0.4 0.4 1.0"/>
+			<origin rpy="0 0 0" xyz="0 0 0"/>
+			<mass value="0.02"/>
+			<inertia ixx="1e-05" ixy="0" ixz="0" iyy="1e-05" iyz="0" izz="1e-05"/>
+		</inertial>
+		<visual>
+			<origin rpy="0 0 0" xyz="0 0 0"/>
+			<geometry>
+				<box size="0.010 0.025 0.080"/>
+			</geometry>
+			<material name="GripperFinger">
+				<color rgba="0.55 0.55 0.55 1.0"/>
 			</material>
 		</visual>
-		<collision>
-			<origin rpy="0 0 0" xyz="0 0 0"/>
-			<geometry>
-				<mesh filename="package://robot_arm/meshes/hande/finger_1_collision.dae" scale="1.0 1.0 1.0"/>
-			</geometry>
-		</collision>
-	</link>
-	<!-- Right finger (mimic of left — Gazebo drives this automatically) -->
-	<joint name="hande_right_finger_joint" type="prismatic">
-		<parent link="hand_e_link"/>
-		<child link="hande_right_finger"/>
-		<origin rpy="0 0 0" xyz="0 0 0.099"/>
-		<axis xyz="1 0 0"/>
-		<limit effort="130" lower="0" upper="0.025" velocity="0.15"/>
-		<mimic joint="hande_left_finger_joint" multiplier="1.0" offset="0.0"/>
-	</joint>
-	<link name="hande_right_finger">
-		<inertial>
-			<origin rpy="0 0 0" xyz="-0.02262 0.00759 0.00738"/>
-			<mass value="0.05"/>
-			<inertia ixx="1e-04" ixy="0" ixz="0" iyy="1e-04" iyz="0" izz="1e-04"/>
-		</inertial>
-		<visual>
-			<origin rpy="0 0 0" xyz="0 0 0"/>
-			<geometry>
-				<mesh filename="package://robot_arm/meshes/hande/finger_2.dae" scale="1.0 1.0 1.0"/>
-			</geometry>
-			<material name="HandE_Gray">
-				<color rgba="0.4 0.4 0.4 1.0"/>
-			</material>
-		</visual>
-		<collision>
-			<origin rpy="0 0 0" xyz="0 0 0"/>
-			<geometry>
-				<mesh filename="package://robot_arm/meshes/hande/finger_2_collision.dae" scale="1.0 1.0 1.0"/>
-			</geometry>
-		</collision>
 	</link>
 	<!-- TCP frame (gripper tip center) -->
@@ -454,18 +446,18 @@
 		</sensor>
 	</gazebo>
-	<!-- Gripper finger physics for grasping -->
+	<!-- Gripper finger physics: disable gravity on both fingers and the
+	     palm so the prismatic left finger never gets dragged by any small
+	     gravity component (axis is +X / horizontal in palm frame, but when
+	     the arm tilts the world-frame gravity gains an X component which
+	     would otherwise bias the joint). No friction tags — collision is
+	     disabled on fingers anyway. -->
+	<gazebo reference="hand_e_link">
+		<gravity>false</gravity>
+	</gazebo>
 	<gazebo reference="hande_left_finger">
-		<mu1>1.0</mu1>
-		<mu2>1.0</mu2>
-		<kp>1000000.0</kp>
-		<kd>1.0</kd>
-		<minDepth>0.001</minDepth>
+		<gravity>false</gravity>
 	</gazebo>
 	<gazebo reference="hande_right_finger">
-		<mu1>1.0</mu1>
-		<mu2>1.0</mu2>
-		<kp>1000000.0</kp>
-		<kd>1.0</kd>
-		<minDepth>0.001</minDepth>
+		<gravity>false</gravity>
 	</gazebo>
 	<!-- ==================== ros2_control ==================== -->
@@ -523,14 +515,13 @@
 			<state_interface name="velocity"/>
 		</joint>
-		<!-- Gripper joints (prismatic) -->
+		<!-- Gripper joint (left finger only — right finger is a fixed link). -->
 		<joint name="hande_left_finger_joint">
 			<command_interface name="position">
-				<param name="min">0</param>
-				<param name="max">0.025</param>
-			</command_interface>
-			<state_interface name="position"/>
-			<state_interface name="velocity"/>
-		</joint>
-		<!-- hande_right_finger_joint: mimic of left, driven by Gazebo physics (no ros2_control interface) -->
+				<param name="min">0.0</param>
+				<param name="max">0.030</param>
+			</command_interface>
+			<state_interface name="position"/>
+			<state_interface name="velocity"/>
+		</joint>
 	</ros2_control>
 	<!-- ==================== Gazebo Sim ROS2 Control Plugin ==================== -->
