Commit message: Add WASD teleoperation node and update setup for Husky robot
- Introduced a new `wasd_teleop.py` script for keyboard-based teleoperation of the Husky robot, allowing control via WASD keys.
- Updated `setup.py` to include the new teleoperation node in the package entry points.
- Created a configuration file `husky_gz_bridge.yaml` to extend the existing bridge with mobile-base topics for better integration with the simulation environment.
- Modified `husky_test.launch.py` to utilize the new bridge configuration and added a static transform publisher for improved frame management in the simulation.
- Updated the URDF file to support dynamic behavior for the Husky robot, allowing it to operate as a free body in the simulation environment.

File: robot_arm/urdf/husky_robocot.urdf.xacro (robot description, xacro)
@@ -20,4 +20,7 @@
 	<!-- Force standalone=false in the included m1013 URDF -->
 	<xacro:arg name="standalone" default="false"/>
+	<!-- mobile=false: Husky fixed to world (F1.4 sanity)
+	     mobile=true:  Husky is a free body; DiffDrive plugin drives wheels via /cmd_vel -->
+	<xacro:arg name="mobile" default="true"/>
 	<!-- ==================== Husky dimensions ==================== -->
 	<xacro:property name="husky_length" value="0.99"/>
@@ -37,11 +40,20 @@
 	<xacro:property name="reservoir_lz"  value="0.2"/>
 	<xacro:property name="reservoir_wall" value="0.01"/>
-	<!-- ==================== World root (TEMP — F2 will remove for free base) ==================== -->
-	<link name="world"/>
-	<joint name="world_to_husky" type="fixed">
-		<origin xyz="0 0 0" rpy="0 0 0"/>
-		<parent link="world"/>
-		<child link="husky_base_link"/>
-	</joint>
+	<!-- ==================== World root ==================== -->
+	<!-- mobile=false: keep Husky fixed to world (debug/sanity).
+	     mobile=true:  Husky is the URDF root; world->husky_base_link is published
+	     dynamically by the DiffDrive plugin via odom. -->
+	<xacro:if value="$(arg mobile)">
+		<!-- No world joint; husky_base_link is the URDF root.
+		     The launch file publishes a static world->odom TF (identity). -->
+	</xacro:if>
+	<xacro:unless value="$(arg mobile)">
+		<link name="world"/>
+		<joint name="world_to_husky" type="fixed">
+			<origin xyz="0 0 0" rpy="0 0 0"/>
+			<parent link="world"/>
+			<child link="husky_base_link"/>
+		</joint>
+	</xacro:unless>
 	<!-- ==================== Husky body ==================== -->
 	<link name="husky_base_link">
@@ -235,3 +247,27 @@
 		</collision>
 	</link>
+	<!-- ==================== DiffDrive (skid-steer 4-wheel) ==================== -->
+	<!-- Subscribes ignition.msgs.Twist on /cmd_vel, drives both left wheels and
+	     both right wheels symmetrically. Publishes /odom and /tf. -->
+	<gazebo>
+		<plugin filename="ignition-gazebo-diff-drive-system"
+		        name="ignition::gazebo::systems::DiffDrive">
+			<left_joint>front_left_wheel_joint</left_joint>
+			<left_joint>rear_left_wheel_joint</left_joint>
+			<right_joint>front_right_wheel_joint</right_joint>
+			<right_joint>rear_right_wheel_joint</right_joint>
+			<wheel_separation>${wheel_track}</wheel_separation>
+			<wheel_radius>${wheel_radius}</wheel_radius>
+			<topic>cmd_vel</topic>
+			<odom_topic>odom</odom_topic>
+			<frame_id>odom</frame_id>
+			<child_frame_id>husky_base_link</child_frame_id>
+			<odom_publish_frequency>50</odom_publish_frequency>
+			<tf_topic>/tf</tf_topic>
+			<max_linear_acceleration>2.0</max_linear_acceleration>
+			<max_angular_acceleration>3.0</max_angular_acceleration>
+			<max_linear_velocity>1.0</max_linear_velocity>
+			<max_angular_velocity>1.5</max_angular_velocity>
+		</plugin>
+	</gazebo>
 </robot>

Commit message: Add cotton branch variants and update demo configurations
- Introduced new cotton branch variants: `branch_variant_A_mature_white_01`, `branch_variant_B_mixed_green_01`, `branch_variant_C_mixed_brown_01`, and `branch_variant_D_sparse_green_01`, including their model and SDF files.
- Updated `cotton_demo_bolls.yaml` and `cotton_demo_clusters.yaml` to incorporate new target variants and enhance the cotton harvesting simulation.
- Adjusted configurations for cotton bolls and clusters to improve visual fidelity and realism in the demo environment.
- Enhanced the overall structure and organization of cotton variant assets for better integration and usability in simulations.

File: robot_arm/urdf/husky_robocot.urdf.xacro (robot description, xacro)
@@ -184,10 +184,9 @@
 			</material>
 		</visual>
-		<collision name="floor_collision">
-			<origin xyz="0 0 ${-reservoir_lz/2 + reservoir_wall/2}"/>
-			<geometry>
-				<box size="${reservoir_lx} ${reservoir_ly} ${reservoir_wall}"/>
-			</geometry>
-		</collision>
+		<!-- No floor collision: bolls are dropped via Gazebo set_pose
+		     teleport (not physical drop), and removing the box from
+		     MoveIt's planning_scene means the arm can path freely from
+		     scout into the reservoir-hover pose without false self-
+		     collision flags against the bin walls. -->
 		<!-- Wall +X -->
 		<visual name="wall_xp_visual">
@@ -198,10 +197,4 @@
 			<material name="reservoir_blue"/>
 		</visual>
-		<collision name="wall_xp_collision">
-			<origin xyz="${reservoir_lx/2 - reservoir_wall/2} 0 0"/>
-			<geometry>
-				<box size="${reservoir_wall} ${reservoir_ly} ${reservoir_lz}"/>
-			</geometry>
-		</collision>
 		<!-- Wall -X -->
 		<visual name="wall_xn_visual">
@@ -212,10 +205,4 @@
 			<material name="reservoir_blue"/>
 		</visual>
-		<collision name="wall_xn_collision">
-			<origin xyz="${-reservoir_lx/2 + reservoir_wall/2} 0 0"/>
-			<geometry>
-				<box size="${reservoir_wall} ${reservoir_ly} ${reservoir_lz}"/>
-			</geometry>
-		</collision>
 		<!-- Wall +Y -->
 		<visual name="wall_yp_visual">
@@ -226,10 +213,4 @@
 			<material name="reservoir_blue"/>
 		</visual>
-		<collision name="wall_yp_collision">
-			<origin xyz="0 ${reservoir_ly/2 - reservoir_wall/2} 0"/>
-			<geometry>
-				<box size="${reservoir_lx} ${reservoir_wall} ${reservoir_lz}"/>
-			</geometry>
-		</collision>
 		<!-- Wall -Y -->
 		<visual name="wall_yn_visual">
@@ -240,10 +221,4 @@
 			<material name="reservoir_blue"/>
 		</visual>
-		<collision name="wall_yn_collision">
-			<origin xyz="0 ${-reservoir_ly/2 + reservoir_wall/2} 0"/>
-			<geometry>
-				<box size="${reservoir_lx} ${reservoir_wall} ${reservoir_lz}"/>
-			</geometry>
-		</collision>
 	</link>
 	<!-- ==================== DiffDrive (skid-steer 4-wheel) ==================== -->
